Commit message: Changed Control Args

File: description/robot_core.xacro (robot description, xacro)
@@ -93,5 +93,5 @@
     </link>
     <gazebo reference="left_wheel">
-        <material>Gazebo/Yellow/material
+        <material>Gazebo/Yellow</material>
     </gazebo>
     <!-- RIGHT WHEEL LINK -->
